File: sensor/amp.sch (KiCad schematic (older format))
At the start: 10 parts, among them IC1 49E, IC2 LM358, J1 TO MCU

Commit message: layout for sensor
Parts:
- added unit 1 of IC2
- C1: footprint (none) -> Capacitors_ThroughHole:CP_Radial_D10.0mm_P5.00mm
- C2: footprint (none) -> Capacitors_ThroughHole:CP_Radial_D5.0mm_P2.00mm
- C3: footprint (none) -> Capacitors_ThroughHole:C_Disc_D5.0mm_W2.5mm_P5.00mm
- IC1: footprint (none) -> TO_SOT_Packages_THT:TO-92_Inline_Narrow_Oval
- IC2: footprint (none) -> SMD_Packages:SOIC-8-N
- J1: footprint (none) -> Pin_Headers:Pin_Header_Straight_1x03_Pitch2.54mm
- R1: value 1k -> 1K; footprint (none) -> Resistors_SMD:R_0805
- R2: value 10k -> 10K; footprint (none) -> Resistors_SMD:R_0805
- R3: value 10k -> 4K7; footprint (none) -> Resistors_SMD:R_0805
- R4: footprint (none) -> Resistors_SMD:R_0805
Connections:
- net at IC1.3 (P3): now also IC2.5 (+); no longer IC2.3 (+)
- net at R2.1, R3.2: now also IC2.7; no longer IC2.1
- net at R1.1, R2.2: now also IC2.6 (-); no longer IC2.2 (-)
- net at R3.1: now also J1.1 (P1); no longer J1.2 (P2)
- net at R4.1: now also J1.2 (P2); no longer J1.1 (P1)
- no-connect marks 0 -> 1
Changed lines of the file:
@@
 LIBS:contrib
 LIBS:valves
+LIBS:amp-cache
 EELAYER 25 0
 EELAYER END
@@
 F 0 "IC1" H 750 1150 50  0000 C CNN
 F 1 "49E" V 850 950 50  0000 C CNN
-F 2 "" H 750 950 50  0001 C CNN
+F 2 "TO_SOT_Packages_THT:TO-92_Inline_Narrow_Oval" H 750 950 50  0001 C CNN
 F 3 "" H 750 950 50  0001 C CNN
 	1    750  950
@@
 $Comp
 L LM358 IC2
-U 1 1 59626325
+U 2 1 59626325
 P 1550 1150
 F 0 "IC2" H 1550 1350 50  0000 L CNN
 F 1 "LM358" H 1550 950 50  0000 L CNN
-F 2 "" H 1550 1150 50  0001 C CNN
+F 2 "SMD_Packages:SOIC-8-N" H 1550 1150 50  0001 C CNN
 F 3 "" H 1550 1150 50  0001 C CNN
-	1    1550 1150
-	1    0    0    -1
-$EndComp
-$Comp
-L +5V #PWR?
+	2    1550 1150
+	1    0    0    -1
+$EndComp
+$Comp
+L +5V #PWR01
 U 1 1 59626378
 P 1450 750
-F 0 "#PWR?" H 1450 600 50  0001 C CNN
+F 0 "#PWR01" H 1450 600 50  0001 C CNN
 F 1 "+5V" H 1450 890 50  0000 C CNN
 F 2 "" H 1450 750 50  0001 C CNN
@@
 $EndComp
 $Comp
-L GND #PWR?
+L GND #PWR02
 U 1 1 59626392
 P 1450 2050
-F 0 "#PWR?" H 1450 1800 50  0001 C CNN
+F 0 "#PWR02" H 1450 1800 50  0001 C CNN
 F 1 "GND" H 1450 1900 50  0000 C CNN
 F 2 "" H 1450 2050 50  0001 C CNN
@@
 F 0 "C2" H 1210 1970 50  0000 L CNN
 F 1 "22µ" H 1210 1820 50  0000 L CNN
-F 2 "" H 1200 1900 50  0001 C CNN
+F 2 "Capacitors_ThroughHole:CP_Radial_D5.0mm_P2.00mm" H 1200 1900 50  0001 C CNN
 F 3 "" H 1200 1900 50  0001 C CNN
 	1    1200 1900
@@
 P 1700 1500
 F 0 "R2" V 1780 1500 50  0000 C CNN
-F 1 "10k" V 1700 1500 50  0000 C CNN
-F 2 "" V 1630 1500 50  0001 C CNN
+F 1 "10K" V 1700 1500 50  0000 C CNN
+F 2 "Resistors_SMD:R_0805" V 1630 1500 50  0001 C CNN
 F 3 "" H 1700 1500 50  0001 C CNN
 	1    1700 1500
@@
 P 1200 1650
 F 0 "R1" V 1280 1650 50  0000 C CNN
-F 1 "1k" V 1200 1650 50  0000 C CNN
-F 2 "" V 1130 1650 50  0001 C CNN
+F 1 "1K" V 1200 1650 50  0000 C CNN
+F 2 "Resistors_SMD:R_0805" V 1130 1650 50  0001 C CNN
 F 3 "" H 1200 1650 50  0001 C CNN
 	1    1200 1650
@@
 P 2100 1150
 F 0 "R3" V 2180 1150 50  0000 C CNN
-F 1 "10k" V 2100 1150 50  0000 C CNN
-F 2 "" V 2030 1150 50  0001 C CNN
+F 1 "4K7" V 2100 1150 50  0000 C CNN
+F 2 "Resistors_SMD:R_0805" V 2030 1150 50  0001 C CNN
 F 3 "" H 2100 1150 50  0001 C CNN
 	1    2100 1150
@@
 F 0 "J1" H 3400 1350 50  0000 C CNN
 F 1 "TO MCU" V 3500 1150 50  0000 C CNN
-F 2 "" H 3400 1150 50  0001 C CNN
+F 2 "Pin_Headers:Pin_Header_Straight_1x03_Pitch2.54mm" H 3400 1150 50  0001 C CNN
 F 3 "" H 3400 1150 50  0001 C CNN
 	1    3400 1150
@@
 F 0 "C1" H 2360 1970 50  0000 L CNN
 F 1 "1000µ" H 2360 1820 50  0000 L CNN
-F 2 "" H 2350 1900 50  0001 C CNN
+F 2 "Capacitors_ThroughHole:CP_Radial_D10.0mm_P5.00mm" H 2350 1900 50  0001 C CNN
 F 3 "" H 2350 1900 50  0001 C CNN
 	1    2350 1900
@@
 F 0 "C3" H 2660 1970 50  0000 L CNN
 F 1 "100n" H 2660 1820 50  0000 L CNN
-F 2 "" H 2650 1900 50  0001 C CNN
+F 2 "Capacitors_ThroughHole:C_Disc_D5.0mm_W2.5mm_P5.00mm" H 2650 1900 50  0001 C CNN
 F 3 "" H 2650 1900 50  0001 C CNN
 	1    2650 1900
@@
 	950  850  2700 850
 Wire Wire Line
-	2250 1150 3200 1150
-Wire Wire Line
 	3200 2050 3200 1250
 Connection ~ 2650 2050
 Wire Wire Line
-	2650 2000 2650 2050
+	2650 2050 2650 2000
 Connection ~ 2650 850
 Wire Wire Line
@@
 Connection ~ 2350 2050
 Wire Wire Line
-	2350 2000 2350 2050
+	2350 2050 2350 2000
 Wire Wire Line
 	1200 2000 1200 2050
@@
 F 0 "R4" V 2930 850 50  0000 C CNN
 F 1 "3R3" V 2850 850 50  0000 C CNN
-F 2 "" V 2780 850 50  0001 C CNN
+F 2 "Resistors_SMD:R_0805" V 2780 850 50  0001 C CNN
 F 3 "" H 2850 850 50  0001 C CNN
 	1    2850 850
 	0    1    1    0
 $EndComp
-Wire Wire Line
-	3000 850  3200 850
-Wire Wire Line
-	3200 850  3200 1050
+NoConn ~ 2050 2700
+$Comp
+L LM358 IC2
+U 1 1 59EC36E3
+P 2050 2550
+F 0 "IC2" H 2050 2750 50  0000 L CNN
+F 1 "LM358" H 2050 2350 50  0000 L CNN
+F 2 "SMD_Packages:SOIC-8-N" H 2050 2550 50  0001 C CNN
+F 3 "" H 2050 2550 50  0001 C CNN
+	1    2050 2550
+	1    0    0    -1
+$EndComp
+Wire Wire Line
+	2250 1150 2900 1150
+Wire Wire Line
+	2900 1150 2900 1050
+Wire Wire Line
+	2900 1050 3200 1050
+Wire Wire Line
+	3000 850  3050 850
+Wire Wire Line
+	3050 850  3050 1150
+Wire Wire Line
+	3050 1150 3200 1150
 $EndSCHEMATC
