File: sensor/amp.kicad_pcb (KiCad board)
At the start: 2 copper layers, 10 parts, among them IC1 49E, IC2 LM358, J1 TO MCU

Commit message: Added layout border
Parts:
- moved C1 108.1 mm to (31.4, 48.4)
- moved C2 108.1 mm to (33.7, 33.9)
- moved C3 108.1 mm to (29.7, 41.4)
- moved IC1 108.1 mm to (25.2, 26.4)
- moved IC2 108.1 mm to (26.4, 33.9)
- moved J1 108.1 mm to (36.2, 46.9)
- moved R1 108.1 mm to (31.4, 28.7)
- moved R2 108.1 mm to (33.7, 28.7)
- moved R3 108.1 mm to (36.2, 42.2)
- moved R4 108.1 mm to (32.5, 41.4)
Other:
- board outline added: 16.2 x 32.3 mm
